Commit message: modify launch file

File: techman_robot/tm_description/urdf/tm.gazebo.xacro (robot description, xacro)
@@ -2,5 +2,25 @@
 <robot xmlns:xacro="http://www.ros.org/wiki/xacro">
   <xacro:macro name="tm_arm_gazebo" params="prefix">
-    <!-- nothing to do here at the moment -->
+    <gazebo reference="${prefix}base_link">
+      <selfCollide>true</selfCollide>
+    </gazebo>
+    <gazebo reference="${prefix}shoulder_1_link">
+      <selfCollide>true</selfCollide>
+    </gazebo>
+    <gazebo reference="${prefix}arm_1_link">
+      <selfCollide>true</selfCollide>
+    </gazebo>
+    <gazebo reference="${prefix}arm_2_link">
+      <selfCollide>true</selfCollide>
+    </gazebo>
+    <gazebo reference="${prefix}wrist_1_link">
+      <selfCollide>true</selfCollide>
+    </gazebo>
+    <gazebo reference="${prefix}wrist_2_link">
+      <selfCollide>true</selfCollide>
+    </gazebo>
+    <gazebo reference="${prefix}wrist_3_link">
+      <selfCollide>true</selfCollide>
+    </gazebo>
   </xacro:macro>
 </robot>

File: techman_robot/tm_description/urdf/tm700.urdf.xacro (robot description, xacro)
@@ -1,8 +1,8 @@
 <?xml version="1.0"?>
 <robot xmlns:xacro="http://www.ros.org/wiki/xacro">
+  <!-- transmission -->
   <xacro:include filename="$(find tm_description)/urdf/tm.transmission.xacro" />
-  <xacro:include filename="$(find tm_description)/urdf/tm.gazebo.xacro" />
+  <!-- Mass parameters -->
   <property name="pi" value="3.14159265" />
-  <!-- Mass parameters-->
   <property name="base_mass" value="1.0" />
   <property name="shoulder_mass" value="4.5" />
@@ -52,4 +52,6 @@
   </xacro:macro>
   <xacro:macro name="tm700_robot" params="prefix joint_limited">
+    <!-- transmission prefix -->
+    <xacro:tm_arm_transmission prefix="${prefix}" />
     <link name="${prefix}base_link" >
       <visual>
@@ -270,19 +272,17 @@
       <origin xyz="0.0 0.0 ${ee_length}" rpy="0.0 0.0 0.0" />
     </joint>
-    <xacro:tm_arm_transmission prefix="${prefix}" />
-    <xacro:tm_arm_gazebo prefix="${prefix}" />
     <!-- ROS base to TM 'base_link' Coordinates transform -->
     <link name="${prefix}base"/>
-    <joint name="${prefix}base_link-base" type="fixed">
+    <joint name="${prefix}base-base_link" type="fixed">
       <origin xyz="0 0 0" rpy="0 0 0"/>
-      <parent link="${prefix}base_link"/>
-      <child link="${prefix}base"/>
+      <parent link="${prefix}base"/>
+      <child link="${prefix}base_link"/>
     </joint>
     <!-- Frame coincident with all-zeros TCP on TM controller -->
     <link name="${prefix}tool0"/>
-    <joint name="${prefix}last_link-tool0" type="fixed">
-      <parent link="${prefix}wrist_3_link"/>
+    <joint name="${prefix}tip_link-tool0" type="fixed">
+      <parent link="${prefix}tip_link"/>
       <child link="${prefix}tool0"/>
-      <origin xyz="0.0 0.0 ${ee_length}" rpy="0.0 0.0 0.0" />
+      <origin xyz="0 0 0" rpy="0 0 0"/>
     </joint>
   </xacro:macro>

File: techman_robot/tm_description/urdf/tm700_robot.urdf.xacro (robot description, xacro)
@@ -1,15 +1,17 @@
 <?xml version="1.0"?>
 <robot name="tm700" xmlns:xacro="http://www.ros.org/wiki/xacro">
-  <!-- common stuff -->
+  <xacro:property name="prefix" value="" />
+  <!-- gazebo stuff -->
   <xacro:include filename="$(find tm_description)/urdf/common.gazebo.xacro" />
+  <xacro:include filename="$(find tm_description)/urdf/tm.gazebo.xacro" />
+  <xacro:tm_arm_gazebo prefix="${prefix}" />
   <!-- tm700 -->
   <xacro:include filename="$(find tm_description)/urdf/tm700.urdf.xacro" />
-  <!-- arm -->
-  <xacro:tm700_robot prefix="" joint_limited="false"/>
+  <xacro:tm700_robot prefix="${prefix}" joint_limited="false" />
   <link name="world" />
   <joint name="world_joint" type="fixed">
     <parent link="world" />
-    <child link = "base_link" />
-    <origin xyz="0.0 0.0 0.0" rpy="0.0 0.0 0.0" />
+    <child link="base" />
+    <origin xyz="0 0 0" rpy="0 0 0" />
   </joint>
 </robot>

File: techman_robot/tm_description/urdf/tm700_robot_joint_limited.urdf.xacro (robot description, xacro)
@@ -1,17 +1,17 @@
 <?xml version="1.0"?>
 <robot name="tm700" xmlns:xacro="http://www.ros.org/wiki/xacro">
-  <!-- common stuff -->
-  <!--
+  <xacro:property name="prefix" value="" />
+  <!-- gazebo stuff -->
   <xacro:include filename="$(find tm_description)/urdf/common.gazebo.xacro" />
-  -->
+  <xacro:include filename="$(find tm_description)/urdf/tm.gazebo.xacro" />
+  <xacro:tm_arm_gazebo prefix="${prefix}" />
   <!-- tm700 -->
   <xacro:include filename="$(find tm_description)/urdf/tm700.urdf.xacro" />
-  <!-- arm -->
-  <xacro:tm700_robot prefix="" joint_limited="true"/>
+  <xacro:tm700_robot prefix="${prefix}" joint_limited="true" />
   <link name="world" />
   <joint name="world_joint" type="fixed">
     <parent link="world" />
-    <child link = "base_link" />
-    <origin xyz="0.0 0.0 0.0" rpy="0.0 0.0 0.0" />
+    <child link="base" />
+    <origin xyz="0 0 0" rpy="0 0 0" />
   </joint>
 </robot>
